Commit message: v1

File: tadeo_ecar_description/urdf/gazebo_ignition.xacro (robot description, xacro)
@@ -118,6 +118,7 @@
     </gazebo>
     <!-- Plugin de cámara para Ignition -->
+    <!-- Plugin de cámara para Ignition - MEJORADO -->
     <gazebo reference="camera_link">
-      <sensor name="camera" type="camera">
+      <sensor name="camera_sensor" type="camera">
         <pose>0 0 0 0 0 0</pose>
         <topic>camera</topic>
@@ -140,10 +141,19 @@
             <stddev>0.007</stddev>
           </noise>
+          <distortion>
+            <k1>0.0</k1>
+            <k2>0.0</k2>
+            <k3>0.0</k3>
+            <p1>0.0</p1>
+            <p2>0.0</p2>
+            <center>0.5 0.5</center>
+          </distortion>
         </camera>
       </sensor>
     </gazebo>
     <!-- Plugin de LiDAR para Ignition -->
+    <!-- Plugin de LiDAR para Ignition - MEJORADO -->
     <gazebo reference="lidar_link">
-      <sensor name="lidar" type="gpu_lidar">
+      <sensor name="lidar_sensor" type="gpu_lidar">
         <pose>0 0 0 0 0 0</pose>
         <topic>scan</topic>
@@ -155,6 +165,6 @@
               <samples>720</samples>
               <resolution>1</resolution>
-              <min_angle>-1.570796</min_angle>
-              <max_angle>1.570796</max_angle>
+              <min_angle>-3.141593</min_angle>
+              <max_angle>3.141593</max_angle>
             </horizontal>
             <vertical>

File: tadeo_ecar_description/urdf/tadeo_ecar.urdf.xacro (robot description, xacro)
@@ -2,6 +2,4 @@
 <robot name="tadeo_ecar" xmlns:xacro="http://www.ros.org/wiki/xacro">
   <!-- AGREGAR: parámetro para package path -->
-  <xacro:arg name="pkg_path" default=""/>
-  <xacro:property name="pkg_path" value="$(arg pkg_path)"/>
   <!-- Incluir archivos de componentes -->
   <xacro:include filename="$(find tadeo_ecar_description)/urdf/materials.xacro"/>

File: tadeo_ecar_description/urdf/tadeo_ecar_base.xacro (robot description, xacro)
@@ -14,5 +14,5 @@
         <geometry>
           <!-- CORREGIDO: usar file:// con path absoluto -->
-          <mesh filename="file://${pkg_path}/meshes/chassis/chasis_base.stl" scale="1 1 1"/>
+          <mesh filename="package://tadeo_ecar_description/meshes/chassis/chasis_base.stl" scale="1 1 1"/>
         </geometry>
         <material name="blue"/>
@@ -21,5 +21,5 @@
         <origin xyz="0 0 ${chassis_z_offset}" rpy="0 0 0"/>
         <geometry>
-          <box size="${chassis_length} ${chassis_width} ${chassis_height}"/>
+          <mesh filename="package://tadeo_ecar_description/meshes/chassis/chasis_base.stl" scale="1 1 1"/>
         </geometry>
       </collision>
@@ -44,5 +44,5 @@
         <geometry>
           <!-- CORREGIDO: usar file:// con path absoluto -->
-          <mesh filename="file://${pkg_path}/meshes/chassis/chasis.stl" scale="0.001 0.001 0.001"/>
+          <mesh filename="package://tadeo_ecar_description/meshes/chassis/chasis.stl" scale="0.001 0.001 0.001"/>
         </geometry>
         <material name="red"/>
@@ -51,5 +51,5 @@
         <origin xyz="-0.49 0.39 ${-chassis_z_offset-0.029}" rpy="${pi/2} 0 ${pi}"/>
         <geometry>
-          <box size="1.0 0.6 0.2"/>
+          <mesh filename="package://tadeo_ecar_description/meshes/chassis/chasis.stl" scale="0.001 0.001 0.001"/>
         </geometry>
       </collision>
@@ -67,5 +67,5 @@
       <parent link="base_link"/>
       <child link="camera_link"/>
-      <origin xyz="0.4 0 ${chassis_height + chassis_z_offset + camera_z_offset}" rpy="0 0 0"/>
+      <origin xyz="0.476 0 ${chassis_height + chassis_z_offset + camera_z_offset + 0.15}" rpy="0 0 0"/>
     </joint>
     <!-- Link de cámara -->
@@ -96,5 +96,5 @@
       <parent link="base_link"/>
       <child link="lidar_link"/>
-      <origin xyz="0.15 0 ${chassis_height - 0.03}" rpy="0 0 0"/>
+      <origin xyz="0.6 0 ${chassis_height - chassis_z_offset + lidar_height}" rpy="0 0 0"/>
     </joint>
     <!-- Link de LiDAR -->

File: tadeo_ecar_description/urdf/tadeo_ecar_wheels.xacro (robot description, xacro)
@@ -16,5 +16,5 @@
         <geometry>
           <!-- CORREGIDO: usar file:// con path absoluto -->
-          <mesh filename="file://${pkg_path}/meshes/suspension/suspension.stl" scale="1 1 1"/>
+          <mesh filename="package://tadeo_ecar_description/meshes/suspension/suspension.stl" scale="1 1 1"/>
         </geometry>
         <material name="gray"/>
@@ -23,5 +23,5 @@
         <origin xyz="0 0 ${suspension_z_offset}" rpy="0 ${pi} ${suspension_rotation}"/>
         <geometry>
-          <box size="0.05 0.05 0.1"/>
+         <mesh filename="package://tadeo_ecar_description/meshes/suspension/suspension.stl" scale="1 1 1"/>
         </geometry>
       </collision>
@@ -47,5 +47,5 @@
         <geometry>
           <!-- CORREGIDO: usar file:// con path absoluto -->
-          <mesh filename="file://${pkg_path}/meshes/wheels/wheel.stl" scale="1 1 1"/>
+          <mesh filename="package://tadeo_ecar_description/meshes/wheels/wheel.stl" scale="1 1 1"/>
         </geometry>
         <material name="black"/>
@@ -54,5 +54,5 @@
         <origin xyz="0 0 0" rpy="${pi/2} 0 0"/>
         <geometry>
-          <cylinder radius="${wheel_radius}" length="${wheel_width}"/>
+          <mesh filename="package://tadeo_ecar_description/meshes/wheels/wheel.stl" scale="1 1 1"/>
         </geometry>
       </collision>

Commit message: v1

File: tadeo_ecar_description/urdf/gazebo_ignition.xacro (robot description, xacro)
@@ -36,4 +36,11 @@
         <diffuse>0.3 0.3 0.3 1</diffuse>
         <specular>0.3 0.3 0.3 1</specular>
+      </material>
+    </gazebo>
+    <gazebo reference="imu_link">
+      <material>
+        <ambient>0.0 1.0 0.0 1</ambient>
+        <diffuse>0.0 1.0 0.0 1</diffuse>
+        <specular>0.0 1.0 0.0 1</specular>
       </material>
     </gazebo>
@@ -188,4 +195,55 @@
       </sensor>
     </gazebo>
+    <!-- Plugin de IMU para Ignition -->
+    <gazebo reference="imu_link">
+      <sensor name="imu_sensor" type="imu">
+        <pose>0 0 0 0 0 0</pose>
+        <topic>imu</topic>
+        <update_rate>100</update_rate>
+        <enable_metrics>false</enable_metrics>
+        <imu>
+          <angular_velocity>
+            <x>
+              <noise type="gaussian">
+                <mean>0.0</mean>
+                <stddev>2e-4</stddev>
+              </noise>
+            </x>
+            <y>
+              <noise type="gaussian">
+                <mean>0.0</mean>
+                <stddev>2e-4</stddev>
+              </noise>
+            </y>
+            <z>
+              <noise type="gaussian">
+                <mean>0.0</mean>
+                <stddev>2e-4</stddev>
+              </noise>
+            </z>
+          </angular_velocity>
+          <linear_acceleration>
+            <x>
+              <noise type="gaussian">
+                <mean>0.0</mean>
+                <stddev>1.7e-2</stddev>
+              </noise>
+            </x>
+            <y>
+              <noise type="gaussian">
+                <mean>0.0</mean>
+                <stddev>1.7e-2</stddev>
+              </noise>
+            </y>
+            <z>
+              <noise type="gaussian">
+                <mean>0.0</mean>
+                <stddev>1.7e-2</stddev>
+              </noise>
+            </z>
+          </linear_acceleration>
+        </imu>
+      </sensor>
+    </gazebo>
   </xacro:macro>
 </robot>

File: tadeo_ecar_description/urdf/tadeo_ecar_base.xacro (robot description, xacro)
@@ -13,5 +13,5 @@
         <origin xyz="0 0 ${chassis_z_offset}" rpy="0 0 0"/>
         <geometry>
-          <!-- CORREGIDO: usar file:// con path absoluto -->
+          <!-- NO QUITAR STL - requerido por el usuario -->
           <mesh filename="package://tadeo_ecar_description/meshes/chassis/chasis_base.stl" scale="1 1 1"/>
         </geometry>
@@ -21,4 +21,5 @@
         <origin xyz="0 0 ${chassis_z_offset}" rpy="0 0 0"/>
         <geometry>
+          <!-- NO QUITAR STL - requerido por el usuario -->
           <mesh filename="package://tadeo_ecar_description/meshes/chassis/chasis_base.stl" scale="1 1 1"/>
         </geometry>
@@ -43,5 +44,5 @@
         <origin xyz="-0.49 0.39 ${-chassis_z_offset-0.029}" rpy="${pi/2} 0 ${pi}"/>
         <geometry>
-          <!-- CORREGIDO: usar file:// con path absoluto -->
+          <!-- NO QUITAR STL - requerido por el usuario -->
           <mesh filename="package://tadeo_ecar_description/meshes/chassis/chasis.stl" scale="0.001 0.001 0.001"/>
         </geometry>
@@ -51,4 +52,5 @@
         <origin xyz="-0.49 0.39 ${-chassis_z_offset-0.029}" rpy="${pi/2} 0 ${pi}"/>
         <geometry>
+          <!-- NO QUITAR STL - requerido por el usuario -->
           <mesh filename="package://tadeo_ecar_description/meshes/chassis/chasis.stl" scale="0.001 0.001 0.001"/>
         </geometry>
@@ -121,4 +123,33 @@
       </inertial>
     </link>
+    <!-- Joint para IMU -->
+    <joint name="imu_joint" type="fixed">
+      <parent link="base_link"/>
+      <child link="imu_link"/>
+      <origin xyz="0 0 ${chassis_height + chassis_z_offset + 0.05}" rpy="0 0 0"/>
+    </joint>
+    <!-- Link de IMU -->
+    <link name="imu_link">
+      <visual>
+        <origin xyz="0 0 0" rpy="0 0 0"/>
+        <geometry>
+          <box size="0.02 0.02 0.01"/>
+        </geometry>
+        <material name="green"/>
+      </visual>
+      <collision>
+        <origin xyz="0 0 0" rpy="0 0 0"/>
+        <geometry>
+          <box size="0.02 0.02 0.01"/>
+        </geometry>
+      </collision>
+      <inertial>
+        <origin xyz="0 0 0" rpy="0 0 0"/>
+        <mass value="0.01"/>
+        <inertia ixx="0.0001" ixy="0.0" ixz="0.0"
+                 iyy="0.0001" iyz="0.0"
+                 izz="0.0001"/>
+      </inertial>
+    </link>
   </xacro:macro>
 </robot>

File: tadeo_ecar_description/urdf/tadeo_ecar_wheels.xacro (robot description, xacro)
@@ -15,5 +15,5 @@
         <origin xyz="0 0 ${suspension_z_offset}" rpy="0 ${pi} ${suspension_rotation}"/>
         <geometry>
-          <!-- CORREGIDO: usar file:// con path absoluto -->
+          <!-- NO QUITAR STL - requerido por el usuario -->
           <mesh filename="package://tadeo_ecar_description/meshes/suspension/suspension.stl" scale="1 1 1"/>
         </geometry>
@@ -23,5 +23,6 @@
         <origin xyz="0 0 ${suspension_z_offset}" rpy="0 ${pi} ${suspension_rotation}"/>
         <geometry>
-         <mesh filename="package://tadeo_ecar_description/meshes/suspension/suspension.stl" scale="1 1 1"/>
+          <!-- NO QUITAR STL - requerido por el usuario -->
+          <mesh filename="package://tadeo_ecar_description/meshes/suspension/suspension.stl" scale="1 1 1"/>
         </geometry>
       </collision>
@@ -46,5 +47,5 @@
         <origin xyz="0 0 0" rpy="${pi/2} 0 0"/>
         <geometry>
-          <!-- CORREGIDO: usar file:// con path absoluto -->
+          <!-- NO QUITAR STL - requerido por el usuario -->
           <mesh filename="package://tadeo_ecar_description/meshes/wheels/wheel.stl" scale="1 1 1"/>
         </geometry>
@@ -54,4 +55,5 @@
         <origin xyz="0 0 0" rpy="${pi/2} 0 0"/>
         <geometry>
+          <!-- NO QUITAR STL - requerido por el usuario -->
           <mesh filename="package://tadeo_ecar_description/meshes/wheels/wheel.stl" scale="1 1 1"/>
         </geometry>
